File: kfchess/kfchess.kicad_sch (KiCad schematic)
At the start: 4 parts, among them U1 XY308-2_54-2P, U2 XY308-2_54-2P, U3 XY308-2_54-2P, U4 Teensy4.1

Commit message: Copied routing for bottom squares
Changed lines of the file:
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@@
 		)
 	)
-	(label "c33"
+	(label "c43"
 		(at 237.49 63.5 180)
 		(fields_autoplaced yes)
@@
 		)
 	)
-	(label "c31"
+	(label "c41"
 		(at 237.49 58.42 180)
 		(fields_autoplaced yes)
@@
 		)
 	)
-	(label "c34"
+	(label "c44"
 		(at 237.49 66.04 180)
 		(fields_autoplaced yes)
@@
 		)
 	)
-	(label "c32"
+	(label "c42"
 		(at 237.49 60.96 180)
 		(fields_autoplaced yes)
