File: ecad/kfchess.kicad_sch (KiCad schematic)
At the start: 4 parts, among them U1 XY308-2_54-2P, U2 XY308-2_54-2P, U3 XY308-2_54-2P, U4 Teensy4.1

Commit message: New layout
Parts:
- removed U1, U2, U3: XY308-2_54-2P, footprint:CONN-TH_XY308-2.54-2P, symbol XY308-2_54-2P:XY308-2_54-2P
- added U1: KF128-5_08-2P, footprint:CONN-TH_P5.08_KF128-5.08-2P, symbol KF128-5_08-2P:KF128-5_08-2P
- added U9: 24_243_2, footprint:CONN-TH_24.243.2, symbol 24_243_2:24_243_2
- U4: footprint teensy:Teensy41_SMT -> teensy:Teensy41
Connections:
- net +5V: now also U1.2
- net GND: now also U1.1
- net at U4.4 (2_OUT2): now also U9.1, U9.2

Commit message: Finished layout
Parts:
- added JP1, JP2: SolderJumper_2_Open, Jumper:SolderJumper-2_P1.3mm_Open_Pad1.0x1.5mm, symbol Jumper:SolderJumper_2_Open
- added U2, U3: DB129VG-5_08-4P-GN-S, footprint:CONN-TH_4P-P5.08_DB129VG-5.08-4P-GN-S, symbol DB129VG-5_08-4P-GN-S:DB129VG-5_08-4P-GN-S
Connections:
- net +5V: now also U2.2, U3.3
- net GND: now also JP1.1 (A), JP2.1 (A), U2.1, U3.4
- net c32: now also U4.32 (40_A16); no longer U4.20 (28_RX7)
- net c33: now also U4.33 (41_A17); no longer U4.21 (29_TX7)
- net c44: now also U4.28 (36_CS); no longer U4.26 (34_RX8)
- net tx_out: now reaches U4.27 (35_TX8)
- net tx_out: now also U3.1
- net jp1: now reaches U4.29 (37_CS)
- net jp1: now also JP1.2 (B)
- net jp2: now reaches U4.5 (3_LRCLK2)
- net jp2: now also JP2.2 (B)
- new net rx_in: U2.4, U4.20 (28_RX7)
- new net rx_out: U3.2, U4.26 (34_RX8)
- new net tx_in: U2.3, U4.21 (29_TX7)
