File: ecad/row.kicad_sch (KiCad schematic)
At the start: 1 part, among them U5 XY308-2_54-8P

Commit message: Finished layout
Parts:
- renumbered U5 to U6
Changed lines of the file:
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@@
 		(dnp no)
 		(fields_autoplaced yes)
-		(property "Reference" "U5"
+		(property "Reference" "U6"
 			(at 107.95 85.09 90)
 			(effects
