File: ecad/square.kicad_sch (KiCad schematic)
At the start: 14 parts, among them Q2 AO3400A

Commit message: New layout
Connections:
- net +5V_em is gone; now on net +5V: D55.1 (K)

Commit message: Finished layout
Parts:
- renumbered D2 to D56, D3 to D57, D4 to D58, D5 to D59, D6 to D60, D7 to D61, D8 to D62, D9 to D63, H4 to H14, Q2 to Q7, R3 to R13, R4 to R14
Changed lines of the file:
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@@
 		(dnp no)
 		(fields_autoplaced yes)
-		(property "Reference" "R3"
+		(property "Reference" "R13"
 			(at 77.47 59.69 90)
 			(effects
@@
 		(dnp no)
 		(fields_autoplaced yes)
-		(property "Reference" "D5"
+		(property "Reference" "D59"
 			(at 232.41 101.6314 0)
 			(effects
@@
 		(dnp no)
 		(fields_autoplaced yes)
-		(property "Reference" "D2"
+		(property "Reference" "D56"
 			(at 118.11 101.6314 0)
 			(effects
@@
 		(dnp no)
 		(fields_autoplaced yes)
-		(property "Reference" "#PWR013"
+		(property "Reference" "#PWR0127"
 			(at 142.24 104.14 0)
 			(effects
@@
 		(dnp no)
 		(fields_autoplaced yes)
-		(property "Reference" "#PWR016"
+		(property "Reference" "#PWR0130"
 			(at 104.14 121.92 0)
 			(effects
@@
 		(dnp no)
 		(fields_autoplaced yes)
-		(property "Reference" "#PWR021"
+		(property "Reference" "#PWR0135"
 			(at 142.24 134.62 0)
 			(effects
@@
 		(dnp no)
 		(fields_autoplaced yes)
-		(property "Reference" "#PWR022"
+		(property "Reference" "#PWR0136"
 			(at 180.34 134.62 0)
 			(effects
@@
 		(dnp no)
 		(fields_autoplaced yes)
-		(property "Reference" "D9"
+		(property "Reference" "D63"
 			(at 232.41 132.1114 0)
 			(effects
@@
 		(dnp no)
 		(fields_autoplaced yes)
-		(property "Reference" "#PWR017"
+		(property "Reference" "#PWR0131"
 			(at 142.24 121.92 0)
 			(effects
@@
 		(dnp no)
 		(fields_autoplaced yes)
-		(property "Reference" "R4"
+		(property "Reference" "R14"
 			(at 87.63 68.5799 0)
 			(effects
@@
 		(dnp no)
 		(fields_autoplaced yes)
-		(property "Reference" "#PWR014"
+		(property "Reference" "#PWR0128"
 			(at 180.34 104.14 0)
 			(effects
@@
 		(dnp no)
 		(fields_autoplaced yes)
-		(property "Reference" "#PWR029"
+		(property "Reference" "#PWR0124"
 			(at 85.09 80.01 0)
 			(effects
@@
 		(dnp no)
 		(fields_autoplaced yes)
-		(property "Reference" "H4"
+		(property "Reference" "H14"
 			(at 204.47 57.1499 0)
 			(effects
@@
 		(dnp no)
 		(fields_autoplaced yes)
-		(property "Reference" "#PWR015"
+		(property "Reference" "#PWR0129"
 			(at 218.44 104.14 0)
 			(effects
@@
 		(dnp no)
 		(fields_autoplaced yes)
-		(property "Reference" "D8"
+		(property "Reference" "D62"
 			(at 194.31 132.1114 0)
 			(effects
@@
 		(dnp no)
 		(fields_autoplaced yes)
-		(property "Reference" "#PWR018"
+		(property "Reference" "#PWR0132"
 			(at 180.34 121.92 0)
 			(effects
@@
 		(dnp no)
 		(fields_autoplaced yes)
-		(property "Reference" "#PWR030"
+		(property "Reference" "#PWR0125"
 			(at 97.79 80.01 0)
 			(effects
@@
 		(dnp no)
 		(fields_autoplaced yes)
-		(property "Reference" "#PWR026"
+		(property "Reference" "#PWR0140"
 			(at 180.34 152.4 0)
 			(effects
@@
 		(dnp no)
 		(fields_autoplaced yes)
-		(property "Reference" "D3"
+		(property "Reference" "D57"
 			(at 156.21 101.6314 0)
 			(effects
@@
 		(dnp no)
 		(fields_autoplaced yes)
-		(property "Reference" "#PWR019"
+		(property "Reference" "#PWR0133"
 			(at 218.44 121.92 0)
 			(effects
@@
 		(dnp no)
 		(fields_autoplaced yes)
-		(property "Reference" "#PWR024"
+		(property "Reference" "#PWR0138"
 			(at 104.14 152.4 0)
 			(effects
@@
 		(dnp no)
 		(fields_autoplaced yes)
-		(property "Reference" "#PWR012"
+		(property "Reference" "#PWR0126"
 			(at 104.14 104.14 0)
 			(effects
@@
 		(dnp no)
 		(fields_autoplaced yes)
-		(property "Reference" "D7"
+		(property "Reference" "D61"
 			(at 156.21 132.1114 0)
 			(effects
@@
 		(dnp no)
 		(fields_autoplaced yes)
-		(property "Reference" "D4"
+		(property "Reference" "D58"
 			(at 194.31 101.6314 0)
 			(effects
@@
 		(dnp no)
 		(fields_autoplaced yes)
-		(property "Reference" "D6"
+		(property "Reference" "D60"
 			(at 118.11 132.1114 0)
 			(effects
@@
 		(dnp no)
 		(fields_autoplaced yes)
-		(property "Reference" "#PWR027"
+		(property "Reference" "#PWR0141"
 			(at 218.44 152.4 0)
 			(effects
@@
 		(dnp no)
 		(fields_autoplaced yes)
-		(property "Reference" "#PWR025"
+		(property "Reference" "#PWR0139"
 			(at 142.24 152.4 0)
 			(effects
@@
 		(dnp no)
 		(fields_autoplaced yes)
-		(property "Reference" "#PWR023"
+		(property "Reference" "#PWR0137"
 			(at 218.44 134.62 0)
 			(effects
@@
 		(dnp no)
 		(fields_autoplaced yes)
-		(property "Reference" "#PWR028"
+		(property "Reference" "#PWR0123"
 			(at 97.79 52.07 0)
 			(effects
@@
 		(dnp no)
 		(fields_autoplaced yes)
-		(property "Reference" "Q2"
+		(property "Reference" "Q7"
 			(at 101.6 64.7699 0)
 			(effects
@@
 		(dnp no)
 		(fields_autoplaced yes)
-		(property "Reference" "#PWR020"
+		(property "Reference" "#PWR0134"
 			(at 104.14 134.62 0)
 			(effects
