File: ecad/kfchess.kicad_pcb (KiCad board)
At the start: 2 copper layers, 260 x 220 mm, 232 parts, among them Q1 AO3400A, Q10 AO3400A, Q11 AO3400A, Q12 AO3400A, Q13 AO3400A, Q14 AO3400A, Q15 AO3400A, Q16 AO3400A, Q2 AO3400A, Q3 AO3400A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

Commit message: Switched to new board shape
Routing:
- net +5V: track 2604.4 -> 2150.8 mm, vias 8 -> 0
- net +5V_em: track 1570.8 -> 1160.7 mm, vias 27 -> 26
- net /s41: track 362.1 -> 76.9 mm, vias 2 -> 1
- net /c41: track 314.0 -> 37.0 mm, vias 2 -> 0
- net /s31: track 345.7 -> 76.9 mm, vias 2 -> 1
- net /c31: track 288.3 -> 36.7 mm, vias 2 -> 0
- net /c42: track 261.0 -> 36.0 mm, vias 2 -> 0
- net /c21: track 256.3 -> 37.2 mm
- net /leds: track 232.2 -> 14.2 mm
- net /s21: track 287.2 -> 76.9 mm, vias 2 -> 1
- net /s11: track 285.4 -> 76.9 mm, vias 2 -> 1
- net /c11: track 226.6 -> 36.8 mm
- net /c32: track 220.2 -> 36.0 mm, vias 2 -> 0
- net /row1/square1/em_n: track 366.6 -> 187.5 mm, vias 3 -> 0
- net /row1/square3/em_n: track 261.8 -> 83.4 mm, vias 3 -> 2
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Other:
- board size 260 x 220 mm -> 240 x 240 mm

Commit message: New layout
Parts:
- removed U2, U3: XY308-2_54-2P, footprint:CONN-TH_XY308-2.54-2P
- added U9: 24_243_2, footprint:CONN-TH_24.243.2, F.Cu at (269.4, 62.1)
- U1: value XY308-2_54-2P -> KF128-5_08-2P; footprint footprint:CONN-TH_XY308-2.54-2P -> footprint:CONN-TH_P5.08_KF128-5.08-2P; moved to F.Cu
- U4: footprint teensy:Teensy41_SMT -> teensy:Teensy41; moved to F.Cu
- moved U5 78.5 mm to (274.4, 85.5), turned to -90 degrees
- moved U1 73.5 mm to (274.0, 48.0)
- moved U6 53.8 mm to (274.4, 136.4), turned to -90 degrees
- moved U4 53.0 mm to (249.1, 30.9), turned to 180 degrees
- moved U7 35.3 mm to (274.4, 183.4), turned to -90 degrees
- moved D115 28.3 mm to (77.7, 247.7)
- moved D117 28.3 mm to (77.7, 222.3)
- moved D124 28.3 mm to (127.7, 247.7)
- moved D126 28.3 mm to (127.7, 222.3)
- moved D16 28.3 mm to (127.7, 97.7)
- moved D43 28.3 mm to (77.7, 147.7)
- moved D45 28.3 mm to (77.7, 122.3)
- moved D52 28.3 mm to (127.7, 147.7)
- moved D54 28.3 mm to (127.7, 122.3)
- moved D7 28.3 mm to (77.7, 97.7)
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Connections:
- D1 pad 1: +5V_em -> +5V
- D10 pad 1: +5V_em -> +5V
- D100 pad 1: +5V_em -> +5V
- D109 pad 1: +5V_em -> +5V
- D118 pad 1: +5V_em -> +5V
- D127 pad 1: +5V_em -> +5V
- D136 pad 1: +5V_em -> +5V
- D19 pad 1: +5V_em -> +5V
- D28 pad 1: +5V_em -> +5V
- D37 pad 1: +5V_em -> +5V
- D46 pad 1: +5V_em -> +5V
- D55 pad 1: +5V_em -> +5V
- D64 pad 1: +5V_em -> +5V
- D73 pad 1: +5V_em -> +5V
- D82 pad 1: +5V_em -> +5V
- D91 pad 1: +5V_em -> +5V
- U1 pad 1: Net-(U4-3_LRCLK2) -> GND
- U1 pad 2: Net-(U4-2_OUT2) -> +5V
- U4 pad 5: Net-(U4-3_LRCLK2) -> unconnected-(U4-3_LRCLK2-Pad5)
- U5 pad 2: +5V_em -> +5V
- U5 pad 4: +5V_em -> +5V
- U5 pad 6: +5V_em -> +5V
- U5 pad 8: +5V_em -> +5V
- U6 pad 2: +5V_em -> +5V
- U6 pad 4: +5V_em -> +5V
- U6 pad 6: +5V_em -> +5V
- U6 pad 8: +5V_em -> +5V
- U7 pad 2: +5V_em -> +5V
- U7 pad 4: +5V_em -> +5V
- U7 pad 6: +5V_em -> +5V
- U7 pad 8: +5V_em -> +5V
- U8 pad 2: +5V_em -> +5V
- U8 pad 4: +5V_em -> +5V
- U8 pad 6: +5V_em -> +5V
- U8 pad 8: +5V_em -> +5V
Routing:
- net +5V: track 2150.8 -> 3311.5 mm, vias 0 -> 26
- net +5V_em: track 1160.7 -> 0.00 mm, vias 26 -> 0

Commit message: Finished layout
Parts:
- added JP1: SolderJumper_2_Open, Jumper:SolderJumper-2_P1.3mm_Open_Pad1.0x1.5mm, B.Cu at (182.2, 34.8)
- added JP2: SolderJumper_2_Open, Jumper:SolderJumper-2_P1.3mm_Open_Pad1.0x1.5mm, B.Cu at (187.2, 34.8)
- added U2: DB129VG-5_08-4P-GN-S, footprint:CONN-TH_4P-P5.08_DB129VG-5.08-4P-GN-S, B.Cu at (67.0, 34.6)
- added U3: DB129VG-5_08-4P-GN-S, footprint:CONN-TH_4P-P5.08_DB129VG-5.08-4P-GN-S, B.Cu at (265.2, 233.9)
- U1, U4, U9: moved to B.Cu
- moved U8 26.6 mm to (265.0, 207.5)
- moved U5 22.9 mm to (265.0, 106.4)
- moved U7 11.0 mm to (265.0, 177.7)
- moved U6 9.45 mm to (265.0, 135.4)
- moved U4 7.46 mm to (249.1, 38.4)
- moved U1 6.20 mm to (274.0, 54.2), turned to -90 degrees
- moved U9 5.50 mm to (269.2, 67.6)
Connections:
- U4 pad 20: /c32 -> /rx_in
- U4 pad 21: /c33 -> /tx_in
- U4 pad 26: /c44 -> /rx_out
- U4 pad 27: unconnected-(U4-35_TX8-Pad27) -> /tx_out
- U4 pad 28: unconnected-(U4-36_CS-Pad28) -> /c44
- U4 pad 29: unconnected-(U4-37_CS-Pad29) -> /jp1
- U4 pad 32: unconnected-(U4-40_A16-Pad32) -> /c32
- U4 pad 33: unconnected-(U4-41_A17-Pad33) -> /c33
- U4 pad 5: unconnected-(U4-3_LRCLK2-Pad5) -> /jp2
Routing:
- net /jp2: track 0.00 -> 85.8 mm
- net /row1/square1/em_n: track 187.5 -> 256.3 mm
- net /row1/square2/em_n: track 136.8 -> 199.3 mm
- net /row3/square1/em_n: track 187.7 -> 245.8 mm
- net /row2/square1/em_n: track 187.6 -> 245.4 mm
- net /row1/square3/em_n: track 83.4 -> 138.4 mm
- net /row4/square3/em_n: track 83.4 -> 136.0 mm
- net /row2/square2/em_n: track 137.0 -> 188.6 mm
- net /row3/square2/em_n: track 137.0 -> 187.1 mm
- net /jp1: track 0.00 -> 49.2 mm
- net /row4/square2/em_n: track 137.0 -> 182.5 mm
- net /row1/square4/em_n: track 35.5 -> 76.1 mm
- net /row2/square3/em_n: track 83.4 -> 123.7 mm
- net Net-(U4-2_OUT2): track 0.00 -> 39.7 mm
- net /s13: track 118.6 -> 156.8 mm
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Other:
- board text added: "+5V"
- board text added: "GND"

Commit message: Finished routing
Routing:
- net +5V: track 3311.5 -> 4187.7 mm, vias 26 -> 27
- net /s41: track 76.9 -> 408.1 mm, vias 1 -> 5
- net /c41: track 37.0 -> 362.4 mm, vias 0 -> 2
- net /s31: track 76.9 -> 362.7 mm, vias 1 -> 3
- net /c42: track 36.0 -> 319.9 mm, vias 0 -> 2
- net /tx_out: track 0.00 -> 278.2 mm
- net /rx_out: track 0.00 -> 271.8 mm
- net /c31: track 36.7 -> 302.1 mm, vias 0 -> 2
- net /c43: track 35.4 -> 279.4 mm, vias 0 -> 3
- net /c32: track 36.0 -> 275.2 mm, vias 0 -> 2
- net /s43: track 118.6 -> 356.4 mm, vias 1 -> 5
- net /c44: track 4.21 -> 238.9 mm, vias 0 -> 2
- net /leds: track 14.2 -> 246.8 mm, vias 1 -> 4
- net /s21: track 76.9 -> 307.3 mm, vias 1 -> 4
- net /c21: track 37.2 -> 254.5 mm, vias 0 -> 2
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
Commit message: Went through and fixed drc
Routing:
- net +5V: track 4187.7 -> 4289.5 mm, vias 27 -> 31
- net /jp2: track 120.4 -> 115.6 mm
- net /c24: track 109.1 -> 110.5 mm
- net GND: vias 130 -> 135
Other:
- board text added: "Real Time Chess Rev B youtube.com/@built-from-scratch"
