File: ecad/edge3/edge1.kicad_pcb (KiCad board)
At the start: 2 copper layers, 240 x 240 mm, 0 parts

Commit message: Added logo to edge4
Other:
- outline, holes or cut-outs redrawn
- board text added: "1"
- board text added: "2"
- board text added: "3"
- board text added: "4"
- board text added: "E"
- board text added: "F"
- board text added: "G"
- board text added: "H"
- board text removed: "5"
- board text removed: "6"
- board text removed: "7"
- board text removed: "8"
- board text removed: "A"
- board text removed: "B"
- board text removed: "C"
- board text removed: "D"
