File: ecad/board/kfchess.kicad_pcb (KiCad board)
At the start: 2 copper layers, 240 x 240 mm, 235 parts, among them Q1 AO3400A, Q10 AO3400A, Q11 AO3400A, Q12 AO3400A, Q13 AO3400A, Q14 AO3400A, Q15 AO3400A, Q16 AO3400A, Q2 AO3400A, Q3 AO3400A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

Commit message: Fixed upside down cross board screw terminals
Parts:
- removed U3: DB129VG-5_08-4P-GN-S, footprint:CONN-TH_4P-P5.08_DB129VG-5.08-4P-GN-S
- added U10: DB128V-5_08-4P-GN-S, footprint:CONN-TH_4P-P5.08_DIBO_DB128V-5.08, B.Cu at (66.9, 34.7)
- U2: value DB129VG-5_08-4P-GN-S -> DB128V-5_08-4P-GN-S; footprint footprint:CONN-TH_4P-P5.08_DB129VG-5.08-4P-GN-S -> footprint:CONN-TH_4P-P5.08_DIBO_DB128V-5.08
- moved U2 281.0 mm to (265.2, 233.8), turned to 90 degrees
Connections:
- U2 pad 1: GND -> /tx_out
- U2 pad 2: +5V -> /rx_out
- U2 pad 3: /tx_in -> +5V
- U2 pad 4: /rx_in -> GND
Routing:
- net /rx_out: track 271.8 -> 273.8 mm
- net +5V: track 4289.5 -> 4291.1 mm
- net /tx_in: track 170.0 -> 169.3 mm
